Commit message: changes for gazebo simulation - wip

File: src/fanuc_moveit_config/config/fanuc_lrmate200id4s.ros2_control.xacro (robot description, xacro)
@@ -2,5 +2,5 @@
 <robot xmlns:xacro="http://www.ros.org/wiki/xacro">
     <xacro:macro name="fanuc_lrmate200id4s_ros2_control" params="name initial_positions_file">
-        <xacro:property name="initial_positions" value="${load_yaml(initial_positions_file)['initial_positions']}"/>
+        <xacro:property name="initial_positions" value="${xacro.load_yaml(initial_positions_file)['initial_positions']}"/>
         <ros2_control name="${name}" type="system">
             <hardware>

File: src/fanuc_moveit_config/config/fanuc_lrmate200id4s.urdf.xacro (robot description, xacro)
@@ -7,3 +7,8 @@
     <xacro:include filename="fanuc_lrmate200id4s.ros2_control.xacro" />
     <xacro:fanuc_lrmate200id4s_ros2_control name="FakeSystem" initial_positions_file="$(arg initial_positions_file)"/>
+    <gazebo>
+        <plugin name="gazebo_ros2_control" filename="libgazebo_ros2_control.so">
+            <robot_sim_type>gazebo_ros2_control/GazeboSystem</robot_sim_type>
+        </plugin>
+    </gazebo>
 </robot>
