Commit message: tried gazebo simulation, but did not work

File: src/fanuc_description/urdf/common_colours.xacro (robot description, xacro)
@@ -1,28 +1,15 @@
 <?xml version="1.0"?>
 <robot xmlns:xacro="http://wiki.ros.org/xacro">
-  <!-- RAL 1021: Rape yellow -->
   <xacro:property name="color_fanuc_yellow"   value="0.96 0.76 0.13 1.0" />
-  <!-- RAL 9002: Grey white -->
   <xacro:property name="color_fanuc_white"    value="0.86 0.85 0.81 1.0" />
-  <!-- RAL 7024: Graphite grey -->
   <xacro:property name="color_fanuc_grey"     value="0.34 0.35 0.36 1.0" />
-  <!-- Roboguide colours -->
-  <!-- #3D3D3D -->
   <xacro:property name="color_fanuc_gray24"   value="${ 61/255} ${ 61/255} ${ 61/255} 1.0" />
-  <!-- #474747 -->
   <xacro:property name="color_fanuc_gray28"   value="${ 71/255} ${ 71/255} ${ 71/255} 1.0" />
-  <!-- #4F4F4F -->
   <xacro:property name="color_fanuc_gray31"   value="${ 79/255} ${ 79/255} ${ 79/255} 1.0" />
-  <!-- #666666 -->
   <xacro:property name="color_fanuc_gray40"   value="${102/255} ${102/255} ${102/255} 1.0" />
-  <!-- #FFFF00 -->
   <xacro:property name="color_fanuc_yellow1"  value="${255/255} ${255/255} ${  0/255} 1.0" />
-  <!-- #BAB0B0 -->
   <xacro:property name="color_fanuc_BAB0B0"   value="${186/255} ${176/255} ${176/255} 1.0" />
-  <!-- #E6E6E6 -->
   <xacro:property name="color_fanuc_E6E6E6"   value="${230/255} ${230/255} ${230/255} 1.0" />
-  <!-- #00FF73: 'collaborative green' -->
   <xacro:property name="color_fanuc_00FF73"   value="${  0/255} ${255/255} ${115/255} 1.0" />
-  <!-- approximations -->
   <xacro:property name="color_fanuc_black"    value="0.15 0.15 0.15 1.0" />
   <xacro:property name="color_fanuc_greyish"  value="0.75 0.75 0.75 1.0" />

File: src/fanuc_description/urdf/lrmate200id4s_macro.xacro (robot description, xacro)
@@ -152,5 +152,5 @@
       <limit effort="0" lower="${radians(-360)}" upper="${radians(360)}" velocity="${radians(900)}" />
     </joint>
-    <!-- ROS-Industrial 'base' frame: base_link to Fanuc World Coordinates transform -->
+    <!-- ROS-Industrial 'base' frame: base_link to Fanuc World Coordinates transform
     <link name="${prefix}base" />
     <joint name="${prefix}base_link-base" type="fixed">
@@ -159,5 +159,5 @@
       <child link="${prefix}base"/>
     </joint>
-    <!-- ROS-Industrial 'flange' frame: attachment point for EEF models -->
+    # ROS-Industrial 'flange' frame: attachment point for EEF models
     <link name="${prefix}flange" />
     <joint name="${prefix}link_6-flange" type="fixed">
@@ -166,5 +166,5 @@
       <child link="${prefix}flange" />
     </joint>
-    <!-- ROS-Industrial 'tool0' frame: all-zeros tool frame -->
+    # ROS-Industrial 'tool0' frame: all-zeros tool frame
     <link name="${prefix}tool0" />
     <joint name="${prefix}flange-tool0" type="fixed">
@@ -172,5 +172,5 @@
       <parent link="${prefix}flange" />
       <child link="${prefix}tool0" />
-    </joint>
+    </joint>-->
   </xacro:macro>
 </robot>

File: src/fanuc_moveit_config/config/fanuc_lrmate200id4s.urdf.xacro (robot description, xacro)
@@ -7,8 +7,3 @@
     <xacro:include filename="fanuc_lrmate200id4s.ros2_control.xacro" />
     <xacro:fanuc_lrmate200id4s_ros2_control name="FakeSystem" initial_positions_file="$(arg initial_positions_file)"/>
-    <gazebo>
-        <plugin name="gazebo_ros2_control" filename="libgazebo_ros2_control.so">
-            <robot_sim_type>gazebo_ros2_control/GazeboSystem</robot_sim_type>
-        </plugin>
-    </gazebo>
 </robot>
