Commit message: added world link to xacro file - stoping work on gazebo sim

File: src/fanuc_description/urdf/lrmate200id4s_macro.xacro (robot description, xacro)
@@ -3,4 +3,5 @@
   <xacro:include filename="$(find moveit_fanuc_description)/urdf/common_materials.xacro"/>
   <xacro:macro name="fanuc_lrmate200id4s" params="prefix">
+    <link name="world"></link>
     <!-- links: main serial chain -->
     <link name="${prefix}base_link">
@@ -110,4 +111,9 @@
     </link>
     <!-- joints: main serial chain -->
+    <joint name="joint_base" type="fixed">
+      <origin xyz="0 0 0" rpy="0 0 0" />
+      <parent link="world" />
+      <child link="base_link" />
+    </joint>
     <joint name="${prefix}joint_1" type="revolute">
       <origin xyz="0 0 0.330" rpy="0 0 0" />

Commit message: added air gripper joint+link(tool0) to urdf

File: src/fanuc_description/urdf/lrmate200id4s_macro.xacro (robot description, xacro)
@@ -179,4 +179,11 @@
       <child link="${prefix}tool0" />
     </joint>-->
+   <!-- ROS-Industrial 'tool0' frame: all-zeros tool frame  -->
+    <link name="${prefix}tool0" />
+    <joint name="${prefix}link_6-tool0" type="fixed">
+      <origin xyz="0.095 0 0" rpy="0 0 0" />
+      <parent link="${prefix}link_6" />
+      <child link="${prefix}tool0" />
+    </joint>
   </xacro:macro>
 </robot>

Commit message: tool0 orientation change urdf

File: src/fanuc_description/urdf/lrmate200id4s_macro.xacro (robot description, xacro)
@@ -182,5 +182,5 @@
     <link name="${prefix}tool0" />
     <joint name="${prefix}link_6-tool0" type="fixed">
-      <origin xyz="0.095 0 0" rpy="0 0 0" />
+      <origin xyz="0 0 0" rpy="3.1415926535 -1.570796327 0" />  <!-- xyz="0.095 0 0" -->
       <parent link="${prefix}link_6" />
       <child link="${prefix}tool0" />
