Commit message: changes in custom fanuc lrmate 200id 4s moveit config -  working

File: src/fanuc_description/urdf/lrmate200id4s.urdf (robot description, URDF)
Before this commit: robot fanuc_lrmate200id4s, 10 links, 9 joints
Links:
- removed link base
- removed link flange
- removed link tool0
Joints:
- removed joint base_link-base
- removed joint flange-tool0
- removed joint link_6-flange

Commit message: changes to urdf + added robot jacobian using pinocchio (now joint 2 vel is correct)

File: src/fanuc_description/urdf/lrmate200id4s.urdf (robot description, URDF)
Before this commit: robot fanuc_lrmate200id4s, 7 links, 6 joints
Links:
- added link tool0
Joints:
- added joint link_6-tool0: type fixed, parent link_6, child tool0, origin xyz=0 0 0 rpy=3.1415926535 -1.570796327 0

Commit message: added fs, ee_mount, rs to urdf + stl - works

File: src/fanuc_description/urdf/lrmate200id4s.urdf (robot description, URDF)
Before this commit: robot fanuc_lrmate200id4s, 8 links, 7 joints
Links:
- added link force_sensor; collision mesh filename=package://moveit_fanuc_description/meshes/collision/fs_15ai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; visual mesh filename=package://moveit_fanuc_description/meshes/visual/fs_15aie.s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
- added link rs_d435i; collision mesh filename=package://moveit_fanuc_description/meshes/collision/rs_d435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; visual mesh filename=package://moveit_fanuc_description/meshes/visual/rs_d435i.s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
- added link rs_mount; collision mesh filename=package://moveit_fanuc_description/meshes/collision/ee_moun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; visual mesh filename=package://moveit_fanuc_description/meshes/visual/ee_mount.s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
Joints:
- added joint eeMount_rs: type fixed, parent rs_mount, child rs_d435i, origin xyz=0 -0.07028 0 rpy=3.1415926535 0 0
- added joint fs_eeMount: type fixed, parent force_sensor, child rs_mount, origin xyz=0 0 -0.005 rpy=0 0 0
- added joint tool0_fs: type fixed, parent tool0, child force_sensor, origin xyz=0 0 0.03052 rpy=3.1415926535 0 -1.570796327

Commit message: axis limit update

File: src/fanuc_description/urdf/lrmate200id4s.urdf (robot description, URDF)
Before this commit: robot fanuc_lrmate200id4s, 11 links, 10 joints
Joints:
- joint joint_3: limit lower=-1.2042771838760873 upper=3.5779249665883754 effort=0 velocity=9.075712110370514 -> lower=-2.13436314 upper=4.88692191 effort=0 velocity=9.075712110370514
